Commit message: added angle conversion services

File: install/robot_description/share/robot_description/urdf/ur5.urdf.xacro (robot description, xacro)
@@ -70,4 +70,10 @@
   </xacro:macro>
   <xacro:macro name="ur5_robot" params="prefix joint_limited">
+    <link name="world"/>
+    <joint name="virtual_joint" type="fixed"> <!--defining the joint that fixes the base of the arm to the ground-->
+      <parent link="world"/>
+      <child link="base_link"/>
+      <origin rpy="0 0 0" xyz="0 0 0"/>
+    </joint>
     <link name="${prefix}base_link" >
       <visual>
