Commit message: added so101 to sim

File: install/robot_description/share/robot_description/so-101/so101.gazebo.xacro (robot description, xacro)
@@ -1,10 +1,8 @@
 <?xml version="1.0"?>
 <robot xmlns:xacro="http://www.ros.org/wiki/xacro" name="so101">
-  <xacro:macro name="so101_gazebo">
-    <gazebo>
-      <plugin filename="gz_ros2_control-system" name="gz_ros2_control::GazeboSimROS2ControlPlugin">
-        <!--<parameters>$(find robot_controller)/config/ur5_controllers.yaml</parameters>-->
-      </plugin>
-    </gazebo>
-  </xacro:macro>
+  <gazebo>
+    <plugin filename="gz_ros2_control-system" name="gz_ros2_control::GazeboSimROS2ControlPlugin">
+      <parameters>$(find robot_controller)/config/so101_controllers.yaml</parameters>
+    </plugin>
+  </gazebo>
 </robot>

File: install/robot_description/share/robot_description/so-101/so101.urdf.xacro (robot description, xacro)
@@ -12,4 +12,10 @@
     <color rgba="0.1 0.1 0.1 1.0"/>
   </material>
+  <link name="world"/> <!--defining link to pin arm to the ground-->
+  <joint name="virtual_joint" type="fixed">
+    <parent link="world"/>
+    <child link="base_link"/>
+    <origin rpy="0 0 0" xyz="0 0 0"/>
+  </joint>
   <!-- Link base -->
   <link name="base_link">
